Commit message: fix urdf

File: AizuSpiderSS.urdf (robot description, URDF)
Before this commit: robot AizuSpiderSS, 24 links, 23 joints
Links:
- added link ARM_CAMERA
- added link FRONT_CAMERA
Joints:
- added joint ARM_CAMERA_tf: type fixed, parent HAND, child ARM_CAMERA, origin xyz=0.0 0.0 0.1055 rpy=0 0 3.14159265358979
- added joint FRONT_CAMERA_tf: type fixed, parent CHASSIS, child FRONT_CAMERA, origin xyz=0.25470 0 0.13550 rpy=0 1.57079632679490 0
